Commit message: Updated a more real road.

File: seat_car_description/urdf/road.xacro (robot description, xacro)
@@ -12,5 +12,5 @@
         <origin xyz="0 0 0" rpy="0 0 0"/>
         <geometry>
-          <box size="1 1 0.02"/>
+          <box size="5 5 0.02"/>
         </geometry>
         <material name="green"/>
@@ -19,5 +19,5 @@
         <origin xyz="0 0 0" rpy="0 0 0"/>
         <geometry>
-          <box size="1 1 0.02"/>
+          <box size="5 5 0.02"/>
         </geometry>
       </collision>

File: seat_car_description/urdf/road_env.xacro (robot description, xacro)
@@ -1,5 +1,5 @@
 <robot name="road" xmlns:xacro="http://www.ros.org/wiki/xacro">
   <xacro:include filename="$(find seat_car_description)/urdf/road.xacro" />
-  <xacro:road name="road1" size="1.0">
+  <xacro:road name="road1" size="5.0">
     <origin xyz="0.0 0.0 0.0" rpy="0 0 0"/>
   </xacro:road>
