Commit message: Added the nodes to perform the visual_gps feature in the simulated car launch file. Changed the names of the frames of the GPS camera. Changed the resolution of the GPS camera to 640x480. Added the colors markers for the visual GPS feature.

File: seat_car_description/urdf/car_sensors.xacro (robot description, xacro)
@@ -117,5 +117,5 @@
   </joint>
   <!-- GPS camera -->
-  <link name="gps_camera">
+  <link name="camera">
     <inertial>
       <mass value="0.1600000" />
@@ -139,14 +139,14 @@
     </collision>
   </link>
-  <joint name="camera_board_gps_camera" type="fixed" >
+  <joint name="camera_board_camera" type="fixed" >
     <parent link="camera_board"/>
-    <child link="gps_camera"/>
+    <child link="camera"/>
     <origin xyz="0.019 0 0.0405" rpy="0 0 0"/>
   </joint>
-  <link name="gps_camera_optical">
-  </link>
-  <joint name="gps_camera_gps_camera_optical" type="fixed" >
-    <parent link="gps_camera"/>
-    <child link="gps_camera_optical"/>
+  <link name="camera_optical">
+  </link>
+  <joint name="camera_camera_optical" type="fixed" >
+    <parent link="camera"/>
+    <child link="camera_optical"/>
     <origin xyz="0.0 0 0.0" rpy="0 -1.5707 0"/>
   </joint>

File: seat_car_description/urdf/road.xacro (robot description, xacro)
@@ -48,4 +48,83 @@
       </collision>
     </link>
+    <joint name="road_link_ceiling" type="fixed">
+      <origin xyz="0 0 2.0" rpy="0 0 0" />
+      <parent link="road_link"/>
+      <child link="ceiling" />
+    </joint>
+    <link name="ceiling">
+    </link>
+    <joint name="ceiling_lamp1" type="fixed">
+      <origin xyz="10 10 -0.02" rpy="0 0 0" />
+      <parent link="ceiling"/>
+      <child link="lamp1" />
+    </joint>
+    <link name="lamp1">
+      <inertial>
+        <mass value="0.001"/>
+        <origin xyz="0.0 0.0 0.0" rpy="0 0 0"/>
+        <inertia ixx="0.00001" ixy="0.0" ixz="0.0" iyy="0.00001" iyz="0.0" izz="0.00001" />
+      </inertial>
+      <visual>
+        <origin xyz="0 0 0" rpy="0 0 0"/>
+        <geometry>
+          <box size="2 2 0.02"/>
+        </geometry>
+      </visual>
+      <collision>
+        <origin xyz="0 0 0" rpy="0 0 0"/>
+        <geometry>
+          <box size="2 2 0.02"/>
+        </geometry>
+      </collision>
+    </link>
+    <joint name="ceiling_lamp2" type="fixed">
+      <origin xyz="10 -10 -0.02" rpy="0 0 0" />
+      <parent link="ceiling"/>
+      <child link="lamp2" />
+    </joint>
+    <link name="lamp2">
+      <inertial>
+        <mass value="0.001"/>
+        <origin xyz="0.0 0.0 0.0" rpy="0 0 0"/>
+        <inertia ixx="0.00001" ixy="0.0" ixz="0.0" iyy="0.00001" iyz="0.0" izz="0.00001" />
+      </inertial>
+      <visual>
+        <origin xyz="0 0 0" rpy="0 0 0"/>
+        <geometry>
+          <box size="2 2 0.02"/>
+        </geometry>
+      </visual>
+      <collision>
+        <origin xyz="0 0 0" rpy="0 0 0"/>
+        <geometry>
+          <box size="2 2 0.02"/>
+        </geometry>
+      </collision>
+    </link>
+    <joint name="ceiling_lamp3" type="fixed">
+      <origin xyz="-10 10 -0.02" rpy="0 0 0" />
+      <parent link="ceiling"/>
+      <child link="lamp3" />
+    </joint>
+    <link name="lamp3">
+      <inertial>
+        <mass value="0.001"/>
+        <origin xyz="0.0 0.0 0.0" rpy="0 0 0"/>
+        <inertia ixx="0.00001" ixy="0.0" ixz="0.0" iyy="0.00001" iyz="0.0" izz="0.00001" />
+      </inertial>
+      <visual>
+        <origin xyz="0 0 0" rpy="0 0 0"/>
+        <geometry>
+          <box size="2 2 0.02"/>
+        </geometry>
+      </visual>
+      <collision>
+        <origin xyz="0 0 0" rpy="0 0 0"/>
+        <geometry>
+          <box size="2 2 0.02"/>
+        </geometry>
+      </collision>
+    </link>
   </xacro:macro>
 </root>

Commit message: seat_car_description: - Added alternative camera plugin with right orientation, commented kinect plugin meanwhile. - Separated gps nodes in gps.launch - Commented road spawn, to be done including launch from road_description package

File: seat_car_description/urdf/car_sensors.xacro (robot description, xacro)
@@ -3,4 +3,5 @@
   <!-- Included URDF Files -->
   <xacro:include filename="$(find seat_car_description)/urdf/car_sensors.gazebo" />
+  <xacro:property name="PI" value="3.1415926535897931" />
   <link name="sensor_board">
     <inertial>
@@ -86,5 +87,5 @@
     <parent link="sensor_board"/>
     <child link="imu"/>
-    <origin xyz="0.239 0.02 0.0025" rpy="0 0 1.5707"/>
+    <origin xyz="0.239 0.02 0.0025" rpy="0 0 ${PI/2}"/>
   </joint>
   <!-- RP_LIDAR -->
@@ -114,5 +115,5 @@
     <parent link="sensor_board"/>
     <child link="laser"/>
-    <origin xyz="0.10445 0 0.0333" rpy="0 0 -3.14159"/>
+    <origin xyz="0.10445 0 0.0333" rpy="0 0 -${PI}"/>
   </joint>
   <!-- GPS camera -->
@@ -149,5 +150,5 @@
     <parent link="camera"/>
     <child link="camera_optical"/>
-    <origin xyz="0.0 0 0.0" rpy="0 -1.5707 0"/>
+    <origin xyz="0.0 0 0.0" rpy="0 -${PI/2} 0"/>
   </joint>
   <!-- Creative camera -->
@@ -177,5 +178,5 @@
     <parent link="camera_board"/>
     <child link="camera_link"/>
-    <origin xyz="0.119 0 0.0" rpy="0 1.5707 0"/>
+    <origin xyz="0.119 0 0.0" rpy="0 ${PI/2} 0"/>
   </joint>
   <link name="camera_rgb_frame">
@@ -198,5 +199,5 @@
     <parent link="camera_link"/>
     <child link="camera_rgb_optical_frame"/>
-    <origin xyz="0.0 0 0.0" rpy="1.5707 -1.5707 0"/>
+    <origin xyz="0.0 0 0.0" rpy="${PI/2} -${PI/2} 0"/>
   </joint>
   <link name="camera_depth_optical_frame">
@@ -205,5 +206,19 @@
     <parent link="camera_link"/>
     <child link="camera_depth_optical_frame"/>
-    <origin xyz="0.0 0 0.0" rpy="1.5707 -1.5707 0"/>
+    <origin xyz="0.0 0 0.0" rpy="${PI/2} -${PI/2} 0"/>
+  </joint>
+  <link name="camera_link2">
+  </link>
+  <joint name="camera_board_camera_link2" type="fixed" >
+    <parent link="camera_board"/>
+    <child link="camera_link2"/>
+    <origin xyz="0.119 0 0.0" rpy="0 0 0"/>
+  </joint>
+  <link name="camera_rgb_optical_frame2">
+  </link>
+  <joint name="camera_link_camera_rgb_optical_frame2" type="fixed" >
+    <parent link="camera_link2"/>
+    <child link="camera_rgb_optical_frame2"/>
+    <origin xyz="0 0 0" rpy="-${PI/2} 0 -${PI/2}"/>
   </joint>
 </robot>
