Commit message: Removed the TF prefix (seat_car) from all frames. Added the odometry node with simulated input to the system. Deleted some unnvecessary physical paremeters from the simulated model. Changed the effort of the traction motor. Chnaged the names of some links to coincide with the names of the real robot. Also added some new frames.

File: seat_car_description/urdf/car.xacro (robot description, xacro)
@@ -6,18 +6,4 @@
   <!-- base_footprint is a fictitious link(frame) that is on the ground right below base_link origin,
        navigation stack depends on this frame -->
-  <link name="base_footprint">
-    <inertial>
-      <mass value="0.001" />
-      <origin xyz="0 0 0" rpy="0 0 0"/>
-      <inertia ixx="0.00001" ixy="0.0" ixz="0.0"
-               iyy="0.00001" iyz="0.0"
-               izz="0.00001" />
-    </inertial>
-  </link>
-  <joint name="base_footprint2base_link" type="fixed">
-    <origin xyz="0 0 0.032" rpy="0 0 0" />
-    <parent link="base_footprint"/>
-    <child link="base_link" />
-  </joint>
   <link name="base_link">
     <inertial>
@@ -48,6 +34,5 @@
     <parent link="base_link" />
     <child link="rear_left_wheel_link" />
-    <limit lower="-1000000000000.0" upper="1000000000000.0" effort="0.92" velocity="124"/>
-    <dynamics damping="0.1"/>
+    <limit lower="-1000000000000.0" upper="1000000000000.0" effort="3.0" velocity="124"/>
   </joint>
   <transmission name="tran_rear_left">
@@ -89,6 +74,5 @@
     <parent link="base_link" />
     <child link="rear_right_wheel_link" />
-    <limit lower="-1000000000000.0" upper="1000000000000.0" effort="0.92" velocity="124"/>
-    <dynamics damping="0.1"/>
+    <limit lower="-1000000000000.0" upper="1000000000000.0" effort="3.0" velocity="124"/>
   </joint>
   <transmission name="tran_rear_right">
@@ -158,6 +142,5 @@
     <parent link="front_left_axel_link" />
     <child link="front_left_wheel_link" />
-    <limit lower="-1000000000000.0" upper="1000000000000.0" effort="0.92" velocity="124"/>
-    <dynamics damping="0.1"/>
+    <limit lower="-1000000000000.0" upper="1000000000000.0" effort="3.0" velocity="124"/>
   </joint>
   <transmission name="tran_front_left_wheel">
@@ -227,6 +210,5 @@
     <parent link="front_right_axel_link" />
     <child link="front_right_wheel_link" />
-    <limit lower="-1000000000000.0" upper="1000000000000.0" effort="0.92" velocity="124"/>
-    <dynamics damping="0.1"/>
+    <limit lower="-1000000000000.0" upper="1000000000000.0" effort="3.0" velocity="124"/>
   </joint>
   <transmission name="tran_front_right_wheel">

File: seat_car_description/urdf/car_sensors.xacro (robot description, xacro)
@@ -89,5 +89,5 @@
   </joint>
   <!-- RP_LIDAR -->
-  <link name="rp_lidar">
+  <link name="laser">
     <inertial>
       <mass value="1.8362923" />
@@ -111,7 +111,7 @@
     </collision>
   </link>
-  <joint name="sensor_board_rp_lidar" type="fixed" >
+  <joint name="sensor_board_laser" type="fixed" >
     <parent link="sensor_board"/>
-    <child link="rp_lidar"/>
+    <child link="laser"/>
     <origin xyz="0.10445 0 0.0333" rpy="0 0 -3.14159"/>
   </joint>
@@ -144,13 +144,13 @@
     <origin xyz="0.019 0 0.0405" rpy="0 0 0"/>
   </joint>
-  <link name="gps_camera_view">
-  </link>
-  <joint name="gps_camera_gps_camera_view" type="fixed" >
+  <link name="gps_camera_optical">
+  </link>
+  <joint name="gps_camera_gps_camera_optical" type="fixed" >
     <parent link="gps_camera"/>
-    <child link="gps_camera_view"/>
+    <child link="gps_camera_optical"/>
     <origin xyz="0.0 0 0.0" rpy="0 -1.5707 0"/>
   </joint>
   <!-- Creative camera -->
-  <link name="creative_camera">
+  <link name="camera_link">
     <inertial>
       <mass value="1.3000000" />
@@ -174,15 +174,36 @@
     </collision>
   </link>
-  <joint name="camera_board_creative_camera" type="fixed" >
+  <joint name="camera_board_camera_link" type="fixed" >
     <parent link="camera_board"/>
-    <child link="creative_camera"/>
+    <child link="camera_link"/>
     <origin xyz="0.119 0 0.0" rpy="0 1.5707 0"/>
   </joint>
-  <link name="creative_camera_view">
-  </link>
-  <joint name="creative_camera_creative_camera_view" type="fixed" >
-    <parent link="creative_camera"/>
-    <child link="creative_camera_view"/>
+  <link name="camera_rgb_frame">
+  </link>
+  <joint name="camera_link_camera_rgb_frame" type="fixed" >
+    <parent link="camera_link"/>
+    <child link="camera_rgb_frame"/>
+    <origin xyz="0.0 0 0.0" rpy="0 0 0"/>
+  </joint>
+  <link name="camera_depth_frame">
+  </link>
+  <joint name="camera_link_camera_depth_frame" type="fixed" >
+    <parent link="camera_link"/>
+    <child link="camera_depth_frame"/>
+    <origin xyz="0.0 0 0.0" rpy="0 0 0"/>
+  </joint>
+  <link name="camera_rgb_optical_frame">
+  </link>
+  <joint name="camera_link_camera_rgb_optical_frame" type="fixed" >
+    <parent link="camera_link"/>
+    <child link="camera_rgb_optical_frame"/>
     <origin xyz="0.0 0 0.0" rpy="1.5707 -1.5707 0"/>
   </joint>
+  <link name="camera_depth_optical_frame">
+  </link>
+  <joint name="camera_link_camera_depth_optical_frame" type="fixed" >
+    <parent link="camera_link"/>
+    <child link="camera_depth_optical_frame"/>
+    <origin xyz="0.0 0 0.0" rpy="1.5707 -1.5707 0"/>
+  </joint>
 </robot>

File: seat_car_description/urdf/road.xacro (robot description, xacro)
@@ -1,4 +1,5 @@
 <?xml version="1.0"?>
 <root xmlns:xacro="http://ros.org/wiki/xacro">
+  <xacro:include filename="$(find seat_car_description)/urdf/road.gazebo" />
   <xacro:macro name="road" params="name size *origin">
     <!-- obstacle -->
@@ -12,5 +13,5 @@
         <origin xyz="0 0 0" rpy="0 0 0"/>
         <geometry>
-          <box size="5 5 0.02"/>
+          <box size="10 10 0.02"/>
         </geometry>
         <material name="green"/>
@@ -19,5 +20,5 @@
         <origin xyz="0 0 0" rpy="0 0 0"/>
         <geometry>
-          <box size="5 5 0.02"/>
+          <box size="10 10 0.02"/>
         </geometry>
       </collision>
@@ -47,8 +48,4 @@
       </collision>
     </link>
-    <gazebo reference="road_link">
-    </gazebo>
-    <gazebo reference="road_image">
-    </gazebo>
   </xacro:macro>
 </root>

Commit message: seat_car_description: updated moved urdf files

File: seat_car_description/urdf/car.xacro (robot description, xacro)
@@ -2,246 +2,14 @@
 <robot name="seat_car" xmlns:xacro="http://www.ros.org/wiki/xacro">
   <!-- Included URDF Files -->
-  <xacro:include filename="$(find seat_car_description)/urdf/materials.xacro" />
-  <xacro:include filename="$(find seat_car_description)/urdf/car_sensors.xacro" />
-  <!-- base_footprint is a fictitious link(frame) that is on the ground right below base_link origin,
-       navigation stack depends on this frame -->
-  <link name="base_link">
-    <inertial>
-      <mass value="6" />
-      <origin xyz="0.15971917 0.00000000 0.00197764" />
-      <inertia ixx="0.0067970" ixy="0.0" ixz="-0.0008808"
-               iyy="0.0784672" iyz="0.0"
-               izz="0.0838770" />
-    </inertial>
-    <visual>
-      <origin xyz="0 0 0" rpy="0 0 0" />
-      <geometry>
-        <mesh filename="package://seat_car_description/meshes/chassis.stl"/>
-      </geometry>
-      <material name="Grey" />
-    </visual>
-    <collision>
-      <origin xyz="0 0 0" rpy="0 0 0" />
-      <geometry>
-        <mesh filename="package://seat_car_description/meshes/chassis.stl"/>
-      </geometry>
-    </collision>
-  </link>
-  <joint name="base_link_rear_left_wheel_joint" type="revolute">
-    <origin xyz="0.0 -0.0825 0" rpy="1.5707 0 0" />
-    <axis xyz="0 0 1" />
-    <anchor xyz="0 0 0" />
-    <parent link="base_link" />
-    <child link="rear_left_wheel_link" />
-    <limit lower="-1000000000000.0" upper="1000000000000.0" effort="3.0" velocity="124"/>
-  </joint>
-  <transmission name="tran_rear_left">
-    <type>transmission_interface/SimpleTransmission</type>
-    <joint name="base_link_rear_left_wheel_joint">
-      <hardwareInterface>EffortJointInterface</hardwareInterface>
-    </joint>
-    <actuator name="rear_left_motor">
-      <hardwareInterface>EffortJointInterface</hardwareInterface>
-      <mechanicalReduction>1</mechanicalReduction>
-    </actuator>
-  </transmission>
-  <link name="rear_left_wheel_link">
-    <inertial>
-      <mass value="1" />
-      <origin xyz="0 0 0" rpy="0 0 0" />
-      <inertia  ixx="0.0002946" ixy="0.0" ixz="0.0"
-                iyy="0.0002946" iyz="0.0"
-                izz="0.000494" />
-    </inertial>
-    <visual>
-      <origin xyz="0 0 0" rpy="0 0 0" />
-      <geometry>
-        <mesh filename="package://seat_car_description/meshes/wheel.stl"/>
-      </geometry>
-      <material name="Black" />
-    </visual>
-    <collision>
-      <origin xyz="0 0 0" rpy="0 0 0" />
-      <geometry>
-        <cylinder radius="0.0315" length="0.001"/>
-      </geometry>
-    </collision>
-  </link>
-  <joint name="base_link_rear_right_wheel_joint" type="revolute">
-    <origin xyz="0.0 0.0825 0" rpy="-1.5707 0 0" />
-    <axis xyz="0 0 1" />
-    <anchor xyz="0 0 0" />
-    <parent link="base_link" />
-    <child link="rear_right_wheel_link" />
-    <limit lower="-1000000000000.0" upper="1000000000000.0" effort="3.0" velocity="124"/>
-  </joint>
-  <transmission name="tran_rear_right">
-    <type>transmission_interface/SimpleTransmission</type>
-    <joint name="base_link_rear_right_wheel_joint">
-      <hardwareInterface>EffortJointInterface</hardwareInterface>
-    </joint>
-    <actuator name="rear_right_motor">
-      <hardwareInterface>EffortJointInterface</hardwareInterface>
-      <mechanicalReduction>1</mechanicalReduction>
-    </actuator>
-  </transmission>
-  <link name="rear_right_wheel_link">
-    <inertial>
-      <mass value="1" />
-      <origin xyz="0 0 0" rpy="0 0 0" />
-      <inertia  ixx="0.0002946" ixy="0.0" ixz="0.0"
-                iyy="0.0002946" iyz="0.0"
-                izz="0.0004940" />
-    </inertial>
-    <visual>
-      <origin xyz="0 0 0" rpy="0 0 0" />
-      <geometry>
-        <mesh filename="package://seat_car_description/meshes/wheel.stl"/>
-      </geometry>
-      <material name="Black" />
-    </visual>
-    <collision>
-      <origin xyz="0 0 0" rpy="0 0 0" />
-      <geometry>
-        <cylinder radius="0.0315" length="0.001"/>
-      </geometry>
-    </collision>
-  </link>
-  <joint name="base_link_front_left_axel_joint" type="revolute">
-    <origin xyz="0.260 -0.0825 0" rpy="1.5707 0 0" />
-    <axis xyz="0 1 0" />
-    <anchor xyz="0 0 0" />
-    <parent link="base_link" />
-    <child link="front_left_axel_link" />
-    <limit lower="-1.5707" upper="1.5707" effort="9.6" velocity="5.3"/>
-    <dynamics damping="0.2"/>
-  </joint>
-  <transmission name="tran_front_left_axel">
-    <type>transmission_interface/SimpleTransmission</type>
-    <joint name="base_link_front_left_axel_joint">
-      <hardwareInterface>EffortJointInterface</hardwareInterface>
-    </joint>
-    <actuator name="front_left_axel_motor">
-      <hardwareInterface>EffortJointInterface</hardwareInterface>
-      <mechanicalReduction>1</mechanicalReduction>
-    </actuator>
-  </transmission>
-  <link name="front_left_axel_link">
-    <inertial>
-      <mass value="0.001" />
-      <origin xyz="0 0 0" rpy="0 0 0" />
-      <inertia  ixx="0.00001" ixy="0.0" ixz="0.0"
-                iyy="0.00001" iyz="0.0"
-                izz="0.00001" />
-    </inertial>
-  </link>
-  <joint name="front_left_axel_front_left_wheel_joint" type="revolute">
-    <origin xyz="0.0 0.0 0" rpy="0 0 0" />
-    <axis xyz="0 0 1" />
-    <anchor xyz="0 0 0" />
-    <parent link="front_left_axel_link" />
-    <child link="front_left_wheel_link" />
-    <limit lower="-1000000000000.0" upper="1000000000000.0" effort="3.0" velocity="124"/>
-  </joint>
-  <transmission name="tran_front_left_wheel">
-    <type>transmission_interface/SimpleTransmission</type>
-    <joint name="front_left_axel_front_left_wheel_joint">
-      <hardwareInterface>EffortJointInterface</hardwareInterface>
-    </joint>
-    <actuator name="front_left_wheel_motor">
-      <hardwareInterface>EffortJointInterface</hardwareInterface>
-      <mechanicalReduction>1</mechanicalReduction>
-    </actuator>
-  </transmission>
-  <link name="front_left_wheel_link">
-    <inertial>
-      <mass value="1" />
-      <origin xyz="0 0 0" rpy="0 0 0" />
-      <inertia  ixx="0.0002946" ixy="0.0" ixz="0.0"
-                iyy="0.0002946" iyz="0.0"
-                izz="0.0004940" />
-    </inertial>
-    <visual>
-      <origin xyz="0 0 0" rpy="0 0 0" />
-      <geometry>
-        <mesh filename="package://seat_car_description/meshes/wheel.stl"/>
-      </geometry>
-      <material name="Black" />
-    </visual>
-    <collision>
-      <origin xyz="0 0 0" rpy="0 0 0" />
-      <geometry>
-        <cylinder radius="0.0315" length="0.001"/>
-      </geometry>
-    </collision>
-  </link>
-  <joint name="base_link_front_right_axel_joint" type="revolute">
-    <origin xyz="0.260 0.0825 0" rpy="-1.5707 0 0" />
-    <axis xyz="0 1 0" />
-    <anchor xyz="0 0 0" />
-    <parent link="base_link" />
-    <child link="front_right_axel_link" />
-    <limit lower="-1.5707" upper="1.5707" effort="9.6" velocity="5.3"/>
-    <dynamics damping="0.2"/>
-  </joint>
-  <transmission name="tran_front_right_axel">
-    <type>transmission_interface/SimpleTransmission</type>
-    <joint name="base_link_front_right_axel_joint">
-      <hardwareInterface>EffortJointInterface</hardwareInterface>
-    </joint>
-    <actuator name="front_right_axel_motor">
-      <hardwareInterface>EffortJointInterface</hardwareInterface>
-      <mechanicalReduction>1</mechanicalReduction>
-    </actuator>
-  </transmission>
-  <link name="front_right_axel_link">
-    <inertial>
-      <mass value="0.001" />
-      <origin xyz="0 0 0" rpy="0 0 0" />
-      <inertia  ixx="0.00001" ixy="0.0" ixz="0.0"
-                iyy="0.00001" iyz="0.0"
-                izz="0.00001" />
-    </inertial>
-  </link>
-  <joint name="front_right_axel_front_right_wheel_joint" type="continuous">
-    <origin xyz="0.0 0.0 0" rpy="0 0 0" />
-    <axis xyz="0 0 1" />
-    <anchor xyz="0 0 0" />
-    <parent link="front_right_axel_link" />
-    <child link="front_right_wheel_link" />
-    <limit lower="-1000000000000.0" upper="1000000000000.0" effort="3.0" velocity="124"/>
-  </joint>
-  <transmission name="tran_front_right_wheel">
-    <type>transmission_interface/SimpleTransmission</type>
-    <joint name="front_right_axel_front_right_wheel_joint">
-      <hardwareInterface>EffortJointInterface</hardwareInterface>
-    </joint>
-    <actuator name="front_right_wheel_motor">
-      <hardwareInterface>EffortJointInterface</hardwareInterface>
-      <mechanicalReduction>1</mechanicalReduction>
-    </actuator>
-  </transmission>
-  <link name="front_right_wheel_link">
-    <inertial>
-      <mass value="1" />
-      <origin xyz="0 0 0" rpy="0 0 0" />
-      <inertia  ixx="0.0002946" ixy="0.0" ixz="0.0"
-                iyy="0.0002946" iyz="0.0"
-                izz="0.0004940" />
-    </inertial>
-    <visual>
-      <origin xyz="0 0 0" rpy="0 0 0" />
-      <geometry>
-        <mesh filename="package://seat_car_description/meshes/wheel.stl"/>
-      </geometry>
-      <material name="Black" />
-    </visual>
-    <collision>
-      <origin xyz="0 0 0" rpy="0 0 0" />
-      <geometry>
-        <cylinder radius="0.0315" length="0.001"/>
-      </geometry>
-    </collision>
-  </link>
-  <xacro:include filename="$(find seat_car_description)/urdf/car.gazebo" />
+  <xacro:include filename="$(find seat_car_description)/urdf/include/materials.xacro" />
+  <xacro:include filename="$(find seat_car_description)/urdf/include/platform.xacro" />
+  <xacro:include filename="$(find seat_car_description)/urdf/include/platform.gazebo" />
+  <xacro:include filename="$(find seat_car_description)/urdf/include/sensors.xacro" />
+  <xacro:include filename="$(find seat_car_description)/urdf/include/sensors.gazebo" />
+  <!-- gazebo sensors -->
+  <xacro:include filename="$(find seat_car_description)/urdf/include/sensors/imu.gazebo" />
+  <xacro:include filename="$(find seat_car_description)/urdf/include/sensors/laser.gazebo" />
+  <!--<xacro:include filename="$(find seat_car_description)/urdf/include/sensors/creative_camera.gazebo" />-->
+  <xacro:include filename="$(find seat_car_description)/urdf/include/sensors/front_camera.gazebo" />
+  <xacro:include filename="$(find seat_car_description)/urdf/include/sensors/gps_camera.gazebo" />
 </robot>

File: seat_car_description/urdf/include/platform.xacro (robot description, xacro)
@@ -2,6 +2,4 @@
 <robot name="seat_car" xmlns:xacro="http://www.ros.org/wiki/xacro">
   <!-- Included URDF Files -->
-  <xacro:include filename="$(find seat_car_description)/urdf/materials.xacro" />
-  <xacro:include filename="$(find seat_car_description)/urdf/car_sensors.xacro" />
   <!-- base_footprint is a fictitious link(frame) that is on the ground right below base_link origin,
        navigation stack depends on this frame -->
@@ -244,4 +242,3 @@
     </collision>
   </link>
-  <xacro:include filename="$(find seat_car_description)/urdf/car.gazebo" />
 </robot>

File: seat_car_description/urdf/include/road/road.xacro (robot description, xacro)
@@ -1,5 +1,4 @@
 <?xml version="1.0"?>
 <root xmlns:xacro="http://ros.org/wiki/xacro">
-  <xacro:include filename="$(find seat_car_description)/urdf/road.gazebo" />
   <xacro:macro name="road" params="name size *origin">
     <!-- obstacle -->

File: seat_car_description/urdf/include/road/road_env.xacro (robot description, xacro)
@@ -1,5 +1,7 @@
+<!-- -->
 <robot name="road" xmlns:xacro="http://www.ros.org/wiki/xacro">
-  <xacro:include filename="$(find seat_car_description)/urdf/road.xacro" />
-  <xacro:road name="road1" size="5.0">
+  <xacro:include filename="$(find seat_car_description)/urdf/include/road/road.xacro" />
+  <xacro:include filename="$(find seat_car_description)/urdf/include/road/road.gazebo" />
+  <xacro:road name="road_circle" size="5.0">
     <origin xyz="0.0 0.0 0.0" rpy="0 0 0"/>
   </xacro:road>

File: seat_car_description/urdf/include/sensors.xacro (robot description, xacro)
@@ -2,5 +2,4 @@
 <robot name="seat_car" xmlns:xacro="http://www.ros.org/wiki/xacro">
   <!-- Included URDF Files -->
-  <xacro:include filename="$(find seat_car_description)/urdf/car_sensors.gazebo" />
   <xacro:property name="PI" value="3.1415926535897931" />
   <link name="sensor_board">
