Commit message: seat_car_description: updated model and sensor xacros

File: seat_car_description/urdf/car.xacro (robot description, xacro)
@@ -10,6 +10,6 @@
   <xacro:include filename="$(find seat_car_description)/urdf/include/sensors/imu.gazebo" />
   <xacro:include filename="$(find seat_car_description)/urdf/include/sensors/laser.gazebo" />
-  <!--<xacro:include filename="$(find seat_car_description)/urdf/include/sensors/creative_camera.gazebo" />-->
-  <xacro:include filename="$(find seat_car_description)/urdf/include/sensors/front_camera.gazebo" />
-  <xacro:include filename="$(find seat_car_description)/urdf/include/sensors/gps_camera.gazebo" />
+  <xacro:include filename="$(find seat_car_description)/urdf/include/sensors/front_rgbd_camera.gazebo" />
+  <!--<xacro:include filename="$(find seat_car_description)/urdf/include/sensors/front_rgb_camera.gazebo" />--> <!-- only rgb, no depth-->
+  <xacro:include filename="$(find seat_car_description)/urdf/include/sensors/top_camera.gazebo" />
 </robot>

File: seat_car_description/urdf/include/platform.xacro (robot description, xacro)
@@ -1,9 +1,7 @@
 <?xml version="1.0"?>
 <robot name="seat_car" xmlns:xacro="http://www.ros.org/wiki/xacro">
-  <!-- Included URDF Files -->
   <xacro:property name="PI" value="3.1415926535897931" />
   <xacro:property name="angle_limit" value="${PI/3.0}" />
-  <!-- base_footprint is a fictitious link(frame) that is on the ground right below base_link origin,
-       navigation stack depends on this frame -->
+  <xacro:property name="wheel_width" value="0.001" />
   <link name="base_link">
     <inertial>
@@ -64,5 +62,5 @@
       <origin xyz="0 0 0" rpy="0 0 0" />
       <geometry>
-        <cylinder radius="0.0315" length="0.001"/>
+        <cylinder radius="0.0315" length="${wheel_width}"/>
       </geometry>
     </collision>
@@ -104,5 +102,5 @@
       <origin xyz="0 0 0" rpy="0 0 0" />
       <geometry>
-        <cylinder radius="0.0315" length="0.001"/>
+        <cylinder radius="0.0315" length="${wheel_width}"/>
       </geometry>
     </collision>
@@ -172,5 +170,5 @@
       <origin xyz="0 0 0" rpy="0 0 0" />
       <geometry>
-        <cylinder radius="0.0315" length="0.001"/>
+        <cylinder radius="0.0315" length="${wheel_width}"/>
       </geometry>
     </collision>
@@ -240,5 +238,5 @@
       <origin xyz="0 0 0" rpy="0 0 0" />
       <geometry>
-        <cylinder radius="0.0315" length="0.001"/>
+        <cylinder radius="0.0315" length="${wheel_width}"/>
       </geometry>
     </collision>

File: seat_car_description/urdf/include/sensors.xacro (robot description, xacro)
@@ -25,5 +25,5 @@
     </collision>
   </link>
-  <joint name="base_link_sensor_board" type="fixed" >
+  <joint name="joint_base_link_to_sensor_board" type="fixed" >
     <parent link="base_link"/>
     <child link="sensor_board"/>
@@ -52,5 +52,5 @@
     </collision>
   </link>
-  <joint name="sensor_board_camera_board" type="fixed" >
+  <joint name="joint_sensor_board_to_camera_board" type="fixed" >
     <parent link="sensor_board"/>
     <child link="camera_board"/>
@@ -83,5 +83,5 @@
     </collision>
   </link>
-  <joint name="sensor_board_imu" type="fixed" >
+  <joint name="joint_sensor_board_to_imu" type="fixed" >
     <parent link="sensor_board"/>
     <child link="imu"/>
@@ -111,11 +111,12 @@
     </collision>
   </link>
-  <joint name="sensor_board_laser" type="fixed" >
+  <joint name="joint_sensor_board_to_laser" type="fixed" >
     <parent link="sensor_board"/>
     <child link="laser"/>
     <origin xyz="0.10445 0 0.0333" rpy="0 0 -${PI}"/>
   </joint>
-  <!-- GPS camera -->
-  <link name="camera">
+  <!-- top camera -->
+  <xacro:property name="top_camera_name" value="top_camera" />
+  <link name="${top_camera_name}">
     <inertial>
       <mass value="0.1600000" />
@@ -126,5 +127,5 @@
     </inertial>
     <visual>
-      <origin xyz="0 0 0" rpy="0 0 0"/>
+      <origin xyz="0 0 0" rpy="0 ${PI/2} 0"/>
       <geometry>
         <mesh filename="package://seat_car_description/meshes/gps_camera.stl" />
@@ -133,5 +134,5 @@
     </visual>
     <collision>
-      <origin xyz="0 0 0" rpy="0 0 0"/>
+      <origin xyz="0 0 0" rpy="0 ${PI/2} 0"/>
       <geometry>
         <mesh filename="package://seat_car_description/meshes/gps_camera.stl" />
@@ -139,18 +140,19 @@
     </collision>
   </link>
-  <joint name="camera_board_camera" type="fixed" >
+  <joint name="joint_camera_board_to_${top_camera_name}" type="fixed" >
     <parent link="camera_board"/>
-    <child link="camera"/>
-    <origin xyz="0.019 0 0.0405" rpy="0 0 0"/>
+    <child link="${top_camera_name}"/>
+    <origin xyz="0.019 0 0.0405" rpy="0 -${PI/2} 0"/>
   </joint>
-  <link name="camera_optical">
+  <link name="${top_camera_name}_optical">
   </link>
-  <joint name="camera_camera_optical" type="fixed" >
-    <parent link="camera"/>
-    <child link="camera_optical"/>
-    <origin xyz="0.0 0 0.0" rpy="0 -${PI/2} 0"/>
+  <joint name="joint_${top_camera_name}_to_${top_camera_name}_optical" type="fixed" >
+    <parent link="${top_camera_name}"/>
+    <child link="${top_camera_name}_optical"/>
+    <origin xyz="0.0 0 0.0" rpy="-${PI/2} 0 -${PI/2}"/>
   </joint>
-  <!-- Creative camera -->
-  <link name="camera_link">
+  <!-- front camera -->
+  <xacro:property name="front_camera_name" value="camera" />
+  <link name="${front_camera_name}_link">
     <inertial>
       <mass value="1.3000000" />
@@ -174,49 +176,14 @@
     </collision>
   </link>
-  <joint name="camera_board_camera_link" type="fixed" >
+  <joint name="joint_camera_board_to_${front_camera_name}_link" type="fixed" >
     <parent link="camera_board"/>
-    <child link="camera_link"/>
-    <origin xyz="0.119 0 0.0" rpy="0 ${PI/2} 0"/>
-  </joint>
-  <link name="camera_rgb_frame">
-  </link>
-  <joint name="camera_link_camera_rgb_frame" type="fixed" >
-    <parent link="camera_link"/>
-    <child link="camera_rgb_frame"/>
-    <origin xyz="0.0 0 0.0" rpy="0 0 0"/>
-  </joint>
-  <link name="camera_depth_frame">
-  </link>
-  <joint name="camera_link_camera_depth_frame" type="fixed" >
-    <parent link="camera_link"/>
-    <child link="camera_depth_frame"/>
-    <origin xyz="0.0 0 0.0" rpy="0 0 0"/>
-  </joint>
-  <link name="camera_rgb_optical_frame">
-  </link>
-  <joint name="camera_link_camera_rgb_optical_frame" type="fixed" >
-    <parent link="camera_link"/>
-    <child link="camera_rgb_optical_frame"/>
-    <origin xyz="0.0 0 0.0" rpy="${PI/2} -${PI/2} 0"/>
-  </joint>
-  <link name="camera_depth_optical_frame">
-  </link>
-  <joint name="camera_link_camera_depth_optical_frame" type="fixed" >
-    <parent link="camera_link"/>
-    <child link="camera_depth_optical_frame"/>
-    <origin xyz="0.0 0 0.0" rpy="${PI/2} -${PI/2} 0"/>
-  </joint>
-  <link name="camera_link2">
-  </link>
-  <joint name="camera_board_camera_link2" type="fixed" >
-    <parent link="camera_board"/>
-    <child link="camera_link2"/>
+    <child link="${front_camera_name}_link"/>
     <origin xyz="0.119 0 0.0" rpy="0 0 0"/>
   </joint>
-  <link name="camera_rgb_optical_frame2">
+  <link name="${front_camera_name}_rgb_optical_frame">
   </link>
-  <joint name="camera_link_camera_rgb_optical_frame2" type="fixed" >
-    <parent link="camera_link2"/>
-    <child link="camera_rgb_optical_frame2"/>
+  <joint name="joint_${front_camera_name}_link_to_${front_camera_name}_rgb_optical_frame" type="fixed" >
+    <parent link="${front_camera_name}_link"/>
+    <child link="${front_camera_name}_rgb_optical_frame"/>
     <origin xyz="0 0 0" rpy="-${PI/2} 0 -${PI/2}"/>
   </joint>
