Commit message: seat_car: moved launch files from seat_car_description to seat_car_launch

File: seat_car_description/urdf/include/road/road.xacro (robot description, xacro)
@@ -37,5 +37,5 @@
         <origin xyz="0 0 0" rpy="0 0 0"/>
         <geometry>
-          <mesh filename="package://seat_car_description/urdf/road.dae" scale="${size*8.63} ${size*8.63} ${size*8.63}"/>
+          <mesh filename="package://seat_car_description/urdf/include/road/road.dae" scale="${size*8.63} ${size*8.63} ${size*8.63}"/>
         </geometry>
       </visual>
@@ -43,5 +43,5 @@
         <origin xyz="0 0 0" rpy="0 0 0"/>
         <geometry>
-          <mesh filename="package://seat_car_description/urdf/road.dae" scale="${size*8.63} ${size*8.63} ${size*8.63}"/>
+          <mesh filename="package://seat_car_description/urdf/include/road/road.dae" scale="${size*8.63} ${size*8.63} ${size*8.63}"/>
         </geometry>
       </collision>
