Commit message: seat_car_description: fixed stl meshes format with meshlab. Rotated top camera frame (yaw pi radians)

File: seat_car_description/urdf/include/sensors.xacro (robot description, xacro)
@@ -143,5 +143,5 @@
     <parent link="camera_board"/>
     <child link="${top_camera_name}"/>
-    <origin xyz="0.019 0 0.0405" rpy="0 -${PI/2} 0"/>
+    <origin xyz="0.019 0 0.0405" rpy="0 -${PI/2} ${PI}"/>
   </joint>
   <link name="${top_camera_name}_optical">
