Commit message: road_description: updated box as xacro instead of sdf. With planar movement (cmd_vel, odom)

File: road_description/urdf/materials.xacro (robot description, xacro)
@@ -10,3 +10,6 @@
     <color rgba="1 0 0 1.0"/>
   </material>
+  <material name="orange">
+    <color rgba="0.93 0.44 0.01 1.0"/>
+  </material>
 </root>
