Commit message: road_description: added trafficlight urdf with ARtag and red/green light

File: road_description/urdf/ceiling_balls.xacro (robot description, xacro)
@@ -1,4 +1,4 @@
 <?xml version="1.0"?>
-<robot name="road" xmlns:xacro="http://www.ros.org/wiki/xacro">
+<robot name="ceiling" xmlns:xacro="http://www.ros.org/wiki/xacro">
   <xacro:include filename="$(find road_description)/urdf/ceiling/ball_macro.xacro" />
   <link name="$(arg parent)"/>

File: road_description/urdf/ceiling_panels.xacro (robot description, xacro)
@@ -1,4 +1,4 @@
 <?xml version="1.0"?>
-<robot name="road" xmlns:xacro="http://www.ros.org/wiki/xacro">
+<robot name="ceiling" xmlns:xacro="http://www.ros.org/wiki/xacro">
   <xacro:include filename="$(find road_description)/urdf/ceiling/panel_macro.xacro" />
   <link name="$(arg parent)"/>

File: road_description/urdf/materials.xacro (robot description, xacro)
@@ -16,3 +16,6 @@
     <color rgba="0 0 0 1.0"/>
   </material>
+  <material name="white">
+    <color rgba="0.9 0.9 0.9 1.0"/>
+  </material>
 </root>
