Commit message: road_description: deleted old/duplicated files. Ceiling panels as circles instead of squares. Updated package.xml files: license, mantainers and authors

File: road_description/urdf/ceiling/panel_macro.xacro (robot description, xacro)
@@ -26,5 +26,6 @@
         <origin xyz="0 0 0" rpy="0 0 0"/>
         <geometry>
-          <box size="${width} ${width} ${thick}"/>
+          <!--<box size="${width} ${width} ${thick}"/>-->
+          <cylinder radius="${width/2.0}" length="${thick}"/>
         </geometry>
         <material name="${urdf_color}"/>
@@ -33,5 +34,6 @@
         <origin xyz="0 0 0" rpy="0 0 0"/>
         <geometry>
-          <box size="${width} ${width} ${thick}"/>
+          <!--<box size="${width} ${width} ${thick}"/>-->
+          <cylinder radius="${width/2.0}" length="${thick}"/>
         </geometry>
       </collision>
