Commit message: road_description: modified trafficlight 0 position. Added colors.txt and map.txt files for gps_visual nodes

File: road_description/urdf/circuits/final/road.xacro (robot description, xacro)
@@ -17,5 +17,5 @@
     </collision>
   </link>
-  <xacro:road name="$(arg name)0" parent="$(arg parent)" dae="full" size="12">
+  <xacro:road name="$(arg name)0" parent="$(arg parent)" dae="final" size="12">
     <origin xyz="0 -5.5 0" rpy="0 0 0"/>
   </xacro:road>

File: road_description/urdf/circuits/final/trafficlights.xacro (robot description, xacro)
@@ -9,5 +9,5 @@
                       light_color="green"
                       light_material="Gazebo/GreenGlow">
-    <origin xyz="1.0 -0.5 0" rpy="0 0 ${PI}"/>
+    <origin xyz="0.75 -0.5 0" rpy="0 0 ${PI}"/>
   </xacro:trafficlight>
   <xacro:trafficlight name="trafficlight1"

File: road_description/urdf/circuits/test/trafficlights.xacro (robot description, xacro)
@@ -9,5 +9,5 @@
                       light_color="green"
                       light_material="Gazebo/GreenGlow">
-    <origin xyz="1.0 -0.5 0" rpy="0 0 ${PI}"/>
+    <origin xyz="0.75 -0.5 0" rpy="0 0 ${PI}"/>
   </xacro:trafficlight>
   <xacro:trafficlight name="trafficlight1"
