Commit message: Added 4th purple ceiling panel

File: road_description/urdf/circuits/final/ceiling_balls.xacro (robot description, xacro)
@@ -21,3 +21,9 @@
     <origin xyz="-4.0 0.0 $(arg height)" rpy="0 0 0"/>
   </xacro:ball>
+  <xacro:ball name="ball_purple"
+               parent="$(arg parent)"
+               gazebo_material="Gazebo/Purple"
+               urdf_color="purple">
+    <origin xyz="-4.0 -11.0 $(arg height)" rpy="0 0 0"/>
+  </xacro:ball>
 </robot>

File: road_description/urdf/circuits/final/ceiling_panels.xacro (robot description, xacro)
@@ -21,3 +21,9 @@
     <origin xyz="-4.0 0.0 $(arg height)" rpy="0 0 0"/>
   </xacro:panel>
+  <xacro:panel name="panel_purple"
+               parent="$(arg parent)"
+               gazebo_material="Gazebo/Purple"
+               urdf_color="purple">
+    <origin xyz="-4.0 -11.0 $(arg height)" rpy="0 0 0"/>
+  </xacro:panel>
 </robot>

File: road_description/urdf/materials.xacro (robot description, xacro)
@@ -19,3 +19,6 @@
     <color rgba="0.9 0.9 0.9 1.0"/>
   </material>
+  <material name="purple">
+    <color rgba="0.5 0.0 0.5 1.0"/>
+  </material>
 </root>
