Commit message: road_description: general updates to xacro files

File: road_description/urdf/box/urdf.xacro (robot description, xacro)
@@ -6,5 +6,5 @@
     <link name="base_link">
       <inertial>
-        <mass value="1" />
+        <mass value="100" />
         <origin xyz="0 0 0" />
         <inertia

File: road_description/urdf/ceiling.xacro (robot description, xacro)
@@ -4,5 +4,5 @@
   <link name="$(arg parent)"/>
   <xacro:ceiling name="$(arg name)" parent="$(arg parent)">
-    <origin xyz="0 0 2.0" rpy="0 0 0"/>
+    <origin xyz="0 0 $(arg height)" rpy="0 0 0"/>
   </xacro:ceiling>
 </robot>

File: road_description/urdf/ceiling/ceiling_macro.xacro (robot description, xacro)
@@ -2,6 +2,20 @@
 <root xmlns:xacro="http://ros.org/wiki/xacro">
   <xacro:include filename="$(find road_description)/urdf/materials.xacro" />
-  <xacro:include filename="$(find road_description)/urdf/ceiling/ceiling.gazebo" />
-  <xacro:macro name="ceiling" params="parent:=ceiling_base_link name:=ceiling *origin">
+  <xacro:property name="default_side" value="10.0" />
+  <xacro:property name="default_width" value="2.0" />
+  <xacro:property name="default_thick" value="0.02" />
+  <xacro:macro name="ceiling"
+               params="parent:=ceiling_base_link
+                       name:=ceiling
+                       *origin
+                       x1:=${default_side}
+                       y1:=${default_side}
+                       x2:=${default_side}
+                       y2:=-${default_side}
+                       x3:=-${default_side}
+                       y3:=${default_side}
+                       width:=${default_width}
+                       length:=${default_width}
+                       thick:=${default_thick}">
     <joint name="joint_${name}_parent_to_link" type="fixed">
       <xacro:insert_block name="origin" />
@@ -12,5 +26,5 @@
     </link>
     <joint name="joint_${name}_to_lamp1" type="fixed">
-      <origin xyz="10 10 -0.02" rpy="0 0 0" />
+      <origin xyz="${x1} ${y1} -${thick/2.0}" rpy="0 0 0" />
       <parent link="${name}"/>
       <child link="lamp1" />
@@ -25,5 +39,5 @@
         <origin xyz="0 0 0" rpy="0 0 0"/>
         <geometry>
-          <box size="2 2 0.02"/>
+          <box size="${length} ${width} ${thick}"/>
         </geometry>
         <material name="red"/>
@@ -32,10 +46,10 @@
         <origin xyz="0 0 0" rpy="0 0 0"/>
         <geometry>
-          <box size="2 2 0.02"/>
+          <box size="${length} ${width} ${thick}"/>
         </geometry>
       </collision>
     </link>
     <joint name="joint_${name}_to_lamp2" type="fixed">
-      <origin xyz="10 -10 -0.02" rpy="0 0 0" />
+      <origin xyz="${x2} ${y2} -${thick/2.0}" rpy="0 0 0" />
       <parent link="${name}"/>
       <child link="lamp2" />
@@ -50,5 +64,5 @@
         <origin xyz="0 0 0" rpy="0 0 0"/>
         <geometry>
-          <box size="2 2 0.02"/>
+          <box size="${length} ${width} ${thick}"/>
         </geometry>
         <material name="green" />
@@ -57,10 +71,10 @@
         <origin xyz="0 0 0" rpy="0 0 0"/>
         <geometry>
-          <box size="2 2 0.02"/>
+          <box size="${length} ${width} ${thick}"/>
         </geometry>
       </collision>
     </link>
     <joint name="joint_${name}_to_lamp3" type="fixed">
-      <origin xyz="-10 10 -0.02" rpy="0 0 0" />
+      <origin xyz="${x3} ${y3} -${thick/2.0}" rpy="0 0 0" />
       <parent link="${name}"/>
       <child link="lamp3" />
@@ -75,5 +89,5 @@
         <origin xyz="0 0 0" rpy="0 0 0"/>
         <geometry>
-          <box size="2 2 0.02"/>
+          <box size="${length} ${width} ${thick}"/>
         </geometry>
         <material name="blue" />
@@ -82,8 +96,23 @@
         <origin xyz="0 0 0" rpy="0 0 0"/>
         <geometry>
-          <box size="2 2 0.02"/>
+          <box size="${length} ${width} ${thick}"/>
         </geometry>
       </collision>
     </link>
+    <gazebo>
+      <static>1</static>
+    </gazebo>
+    <gazebo reference="ceiling">
+      <material>Gazebo/Grey</material>
+    </gazebo>
+    <gazebo reference="lamp1">
+      <material>Gazebo/Red</material>
+    </gazebo>
+    <gazebo reference="lamp2">
+      <material>Gazebo/Green</material>
+    </gazebo>
+    <gazebo reference="lamp3">
+      <material>Gazebo/Blue</material>
+    </gazebo>
   </xacro:macro>
 </root>

File: road_description/urdf/circuit_8.xacro (robot description, xacro)
@@ -3,8 +3,18 @@
   <xacro:include filename="$(find road_description)/urdf/roads/road_piece.xacro" />
   <xacro:include filename="$(find road_description)/urdf/roads/road_ground.xacro" />
-  <link name="$(arg parent)"/>
-  <xacro:road_ground name="$(arg name)_ground" parent="$(arg parent)" dae="empty" size="10.0">
-    <origin xyz="1.5 3.5 0" rpy="0 0 0"/>
-  </xacro:road_ground>
+  <link name="$(arg parent)">
+    <inertial>
+      <mass value="100"/>
+      <origin xyz="0 0 0" rpy="0 0 0"/>
+      <inertia ixx="21.33933333" ixy="0" ixz="0" iyy="13.73933333" iyz="0" izz="35.07266667" />
+    </inertial>
+    <collision>
+      <origin xyz="0 0 0" rpy="0 0 0"/>
+      <geometry>
+        <box size="0.01 0.01 0.01"/>
+      </geometry>
+      <material name="red"/>
+    </collision>
+  </link>
   <xacro:road name="$(arg name)1" parent="$(arg parent)" dae="straight">
     <origin xyz="0 0 0" rpy="0 0 0"/>

File: road_description/urdf/circuit_junctions.xacro (robot description, xacro)
@@ -3,8 +3,18 @@
   <xacro:include filename="$(find road_description)/urdf/roads/road_piece.xacro" />
   <xacro:include filename="$(find road_description)/urdf/roads/road_ground.xacro" />
-  <link name="$(arg parent)"/>
-  <xacro:road_ground name="$(arg name)_ground" parent="$(arg parent)" dae="empty" size="12.0">
-    <origin xyz="0 -4.5 0" rpy="0 0 0"/>
-  </xacro:road_ground>
+  <link name="$(arg parent)">
+    <inertial>
+      <mass value="100"/>
+      <origin xyz="0 0 0" rpy="0 0 0"/>
+      <inertia ixx="21.33933333" ixy="0" ixz="0" iyy="13.73933333" iyz="0" izz="35.07266667" />
+    </inertial>
+    <collision>
+      <origin xyz="0 0 0" rpy="0 0 0"/>
+      <geometry>
+        <box size="0.01 0.01 0.01"/>
+      </geometry>
+      <material name="red"/>
+    </collision>
+  </link>
   <xacro:road name="$(arg name)1" parent="$(arg parent)" dae="straight">
     <origin xyz="0 0 0" rpy="0 0 0"/>

File: road_description/urdf/circuit_o.xacro (robot description, xacro)
@@ -3,8 +3,18 @@
   <xacro:include filename="$(find road_description)/urdf/roads/road_piece.xacro" />
   <xacro:include filename="$(find road_description)/urdf/roads/road_ground.xacro" />
-  <link name="$(arg parent)"/>
-  <xacro:road_ground name="$(arg name)_ground" parent="$(arg parent)" dae="empty" size="10.0">
-    <origin xyz="0 2 0" rpy="0 0 0"/>
-  </xacro:road_ground>
+  <link name="$(arg parent)">
+    <inertial>
+      <mass value="100"/>
+      <origin xyz="0 0 0" rpy="0 0 0"/>
+      <inertia ixx="21.33933333" ixy="0" ixz="0" iyy="13.73933333" iyz="0" izz="35.07266667" />
+    </inertial>
+    <collision>
+      <origin xyz="0 0 0" rpy="0 0 0"/>
+      <geometry>
+        <box size="0.01 0.01 0.01"/>
+      </geometry>
+      <material name="red"/>
+    </collision>
+  </link>
   <xacro:road name="$(arg name)1" parent="$(arg parent)" dae="straight" size="1.0">
     <origin xyz="0 0 0" rpy="0 0 0"/>

File: road_description/urdf/cylinder/urdf.xacro (robot description, xacro)
@@ -6,5 +6,5 @@
     <link name="base_link">
       <inertial>
-        <mass value="1" />
+        <mass value="100" />
         <origin xyz="0 0 0" />
         <inertia

File: road_description/urdf/materials.xacro (robot description, xacro)
@@ -13,3 +13,6 @@
     <color rgba="0.93 0.44 0.01 1.0"/>
   </material>
+  <material name="black">
+    <color rgba="0 0 0 1.0"/>
+  </material>
 </root>

File: road_description/urdf/roads/road_ground.xacro (robot description, xacro)
@@ -1,8 +1,7 @@
 <?xml version="1.0"?>
 <root xmlns:xacro="http://ros.org/wiki/xacro">
-  <xacro:include filename="$(find road_description)/urdf/roads/road.gazebo" />
   <xacro:property name="PI" value="3.1415926535897931" />
   <xacro:macro name="road_ground" params="parent:=road_base_link name:=road size:=1.0 dae:=empty thickness:=0.01 *origin">
-    <joint name="joint_${name}_parent_to_link" type="fixed">
+    <joint name="joint_${parent}_to_${name}_link" type="fixed">
       <xacro:insert_block name="origin" />
       <parent link="${parent}"/>
@@ -15,11 +14,4 @@
         <inertia ixx="21.33933333" ixy="0" ixz="0" iyy="13.73933333" iyz="0" izz="35.07266667" />
       </inertial>
-      <visual>
-        <origin xyz="0 0 ${thickness/2}" rpy="0 0 0"/>
-        <geometry>
-          <box size="${size} ${size} ${thickness}"/>
-        </geometry>
-        <material name="green"/>
-      </visual>
       <collision>
         <origin xyz="0 0 ${thickness/2}" rpy="0 0 0"/>
@@ -27,17 +19,13 @@
           <box size="${size} ${size} ${thickness}"/>
         </geometry>
+        <material name="black"/>
       </collision>
     </link>
-    <joint name="joint_${name}_link_to_image" type="fixed">
-      <origin xyz="0 0 ${thickness+0.001}" rpy="${PI/2} 0 -${PI/2}" />
+    <joint name="joint_${name}_link_to_${name}_image" type="fixed">
+      <origin xyz="0 0 ${thickness}" rpy="${PI/2} 0 -${PI/2}" />
       <parent link="${name}_link"/>
       <child link="${name}_image" />
     </joint>
     <link name="${name}_image">
-      <inertial>
-        <mass value="0.001"/>
-        <origin xyz="0 0 0" rpy="0 0 0"/>
-        <inertia ixx="0.00001" ixy="0" ixz="0" iyy="0.00001" iyz="0" izz="0.00001" />
-      </inertial>
       <visual>
         <origin xyz="0 0 0" rpy="0 0 0"/>
@@ -46,11 +34,13 @@
         </geometry>
       </visual>
-      <collision>
-        <origin xyz="0 0 0" rpy="0 0 0"/>
-        <geometry>
-          <mesh filename="package://road_description/urdf/roads/dae/${dae}.dae" scale="${size} 1.0 ${size}"/>
-        </geometry>
-      </collision>
     </link>
+    <gazebo>
+      <static>1</static>
+    </gazebo>
+    <gazebo reference="${name}_link">
+      <material>Gazebo/Black</material>
+    </gazebo>
+    <gazebo reference="${name}_image">
+    </gazebo>
   </xacro:macro>
 </root>

File: road_description/urdf/roads/road_piece.xacro (robot description, xacro)
@@ -1,7 +1,6 @@
 <?xml version="1.0"?>
 <root xmlns:xacro="http://ros.org/wiki/xacro">
-  <xacro:include filename="$(find road_description)/urdf/roads/road.gazebo" />
   <xacro:property name="PI" value="3.1415926535897931" />
-  <xacro:macro name="road" params="parent:=road_base_link name:=road size:=1.0 dae:=straight thickness:=0.02 *origin">
+  <xacro:macro name="road" params="parent:=road_base_link name:=road size:=1.0 dae:=straight height:=0.001 *origin">
     <joint name="joint_${name}_parent_to_link" type="fixed">
       <xacro:insert_block name="origin" />
@@ -10,34 +9,11 @@
     </joint>
     <link name="${name}_link">
-      <!--<inertial>
-        <mass value="100"/>
-        <origin xyz="0 0 ${thickness/2}" rpy="0 0 0"/>
-        <inertia ixx="21.33933333" ixy="0" ixz="0" iyy="13.73933333" iyz="0" izz="35.07266667" />
-      </inertial>
-      <visual>
-        <origin xyz="0 0 ${thickness/2}" rpy="0 0 0"/>
-        <geometry>
-          <box size="${size} ${size} ${thickness}"/>
-        </geometry>
-        <material name="green"/>
-      </visual>
-      <collision>
-        <origin xyz="0 0 ${thickness/2}" rpy="0 0 0"/>
-        <geometry>
-          <box size="${size} ${size} ${thickness}"/>
-        </geometry>
-      </collision>-->
     </link>
     <joint name="joint_${name}_link_to_image" type="fixed">
-      <origin xyz="0 0 ${thickness+0.001}" rpy="${PI/2} 0 -${PI/2}" />
+      <origin xyz="0 0 ${height}" rpy="${PI/2} 0 -${PI/2}" />
       <parent link="${name}_link"/>
       <child link="${name}_image" />
     </joint>
     <link name="${name}_image">
-      <inertial>
-        <mass value="0.001"/>
-        <origin xyz="0 0 0" rpy="0 0 0"/>
-        <inertia ixx="0.00001" ixy="0" ixz="0" iyy="0.00001" iyz="0" izz="0.00001" />
-      </inertial>
       <visual>
         <origin xyz="0 0 0" rpy="0 0 0"/>
@@ -46,11 +22,13 @@
         </geometry>
       </visual>
-      <collision>
-        <origin xyz="0 0 0" rpy="0 0 0"/>
-        <geometry>
-          <mesh filename="package://road_description/urdf/roads/dae/${dae}.dae" scale="${size} 1.0 ${size}"/>
-        </geometry>
-      </collision>
     </link>
+    <gazebo>
+      <static>1</static>
+    </gazebo>
+    <gazebo reference="${name}_link">
+      <material>Gazebo/Black</material>
+    </gazebo>
+    <gazebo reference="${name}_image">
+    </gazebo>
   </xacro:macro>
 </root>

Commit message: seat_car_simulator: updated to match seat-adc rule book v1.2  - updated circuit (name: full): road-track design, trafficlights and obstacle positions  - added color_plugin package to change trafficlight lights with topics/service calls

File: road_description/urdf/box/urdf.xacro (robot description, xacro)
@@ -39,5 +39,5 @@
           <box size="${LENGTH} ${WIDTH} ${HEIGHT}"/>
         </geometry>
-        <material name="orange"/>
+        <material name="grey"/>
       </visual>
     </link>

File: road_description/urdf/circuits/full/road.xacro (robot description, xacro)
@@ -17,6 +17,6 @@
     </collision>
   </link>
-  <xacro:road name="$(arg name)0" parent="$(arg parent)" dae="final_parking" size="13">
-    <origin xyz="-0.5 -6.0 0" rpy="0 0 0"/>
+  <xacro:road name="$(arg name)0" parent="$(arg parent)" dae="full" size="12">
+    <origin xyz="0.0 -5.07 0" rpy="0 0 0"/>
   </xacro:road>
 </robot>

File: road_description/urdf/circuits/full/trafficlights_fixed.xacro (robot description, xacro)
@@ -11,5 +11,5 @@
                       light_material="Gazebo/RedGlow"
                       light_material2="Gazebo/GreenGlow">
-    <origin xyz="1.0 -0.5 0" rpy="0 0 ${PI}"/>
+    <origin xyz="1.05 -0.5 0" rpy="0 0 ${PI}"/>
   </xacro:trafficlight>
   <xacro:trafficlight name="semaphore_start2"
@@ -19,5 +19,5 @@
                       light_material="Gazebo/RedGlow"
                       light_material2="Gazebo/GreenGlow">
-    <origin xyz="-1.0 0.5 0" rpy="0 0 0"/>
+    <origin xyz="-1.05 0.5 0" rpy="0 0 0"/>
   </xacro:trafficlight>
   <xacro:trafficlight name="semaphore_parking1"
@@ -27,5 +27,5 @@
                       light_material="Gazebo/Blue"
                       light_material2="Gazebo/Black">
-    <origin xyz="-1.0 -10.5 0" rpy="0 0 0"/>
+    <origin xyz="1.55 -0.5 0" rpy="0 0 ${PI}"/>
   </xacro:trafficlight>
   <xacro:trafficlight name="semaphore_parking2"
@@ -34,5 +34,5 @@
                       light_color="blue"
                       light_material="Gazebo/Blue">
-    <origin xyz="-6.0 -2.5 0" rpy="0 0 ${PI/2}"/>
+    <origin xyz="-3.1 -0.5 0" rpy="0 0 ${PI}"/>
   </xacro:trafficlight>
 </robot>

File: road_description/urdf/materials.xacro (robot description, xacro)
@@ -22,3 +22,9 @@
     <color rgba="0.5 0.0 0.5 1.0"/>
   </material>
+  <material name="yellow">
+    <color rgba="1.0 1.0 0.0 1.0"/>
+  </material>
+  <material name="grey">
+    <color rgba="0.4 0.4 0.4 1.0"/>
+  </material>
 </root>

File: road_description/urdf/trafficlight/signal_macro.xacro (robot description, xacro)
@@ -1,5 +1,5 @@
 <?xml version="1.0"?>
 <root xmlns:xacro="http://ros.org/wiki/xacro">
-  <xacro:include filename="$(find road_description)/urdf/materials.xacro" />
+  <!--<xacro:include filename="$(find road_description)/urdf/materials.xacro" />-->
   <xacro:property name="PI" value="3.1415926535897931" />
   <xacro:property name="panel_width"    value="0.07" />
@@ -12,9 +12,10 @@
   <xacro:property name="light_height"   value="0.025" />
   <xacro:property name="light_z_offset" value="0.125" />
-  <xacro:macro name="trafficlight"
-               params="name:=trafficlight
+  <xacro:macro name="signal"
+               params="name:=signal
                        parent:=${name}_base_link
                        *origin
-                       tag_dae:=tag47
+                       tag_dae:=tag57
+                       signal_dae:=arrow_left
                        light_color:=red
                        light_material:=Gazebo/RedGlow
@@ -22,4 +23,5 @@
                        ">
     <!-- tag_dae = tag95, tag47, tag74, tag29, tag57 -->
+    <!-- signal_dae = arrow_left, arrow_right -->
     <!-- light_color    = red,            green,            blue,           black -->
     <!-- light_material = Gazebo/RedGlow, Gazebo/GreenGlow, Gazebo/BlueSky, Gazebo/Black -->
@@ -96,5 +98,5 @@
     </link>
     <joint name="joint_${name}_light_link_to_${name}_light_image" type="fixed">
-      <origin xyz="${panel_depth/2.0+delta} 0 ${light_height/2.0+light_z_offset}" rpy="0 0 0" />
+      <origin xyz="${panel_depth/2.0+delta} 0 ${light_height/2.0+light_z_offset}" rpy="0 ${PI} -${PI/2}" />
       <parent link="${name}_light_link"/>
       <child link="${name}_light_image" />
@@ -104,7 +106,6 @@
         <origin xyz="0 0 0" rpy="0 0 0"/>
         <geometry>
-          <box size="0.001 ${light_width} ${light_height}"/>
+          <mesh filename="package://road_description/urdf/trafficlight/dae/${signal_dae}.dae" scale="${light_width} 1.0 ${light_height}"/>
         </geometry>
-        <material name="${light_color}"/>
       </visual>
     </link>
@@ -116,11 +117,4 @@
     <gazebo reference="${name}_light_image">
       <!--<material>${light_material}</material>-->
-      <visual>
-        <plugin name="${name}_color_plugin" filename="libcolor_plugin.so" >
-          <element_name>${name}</element_name>
-          <material>${light_material}</material>
-          <material2>${light_material2}</material2>
-        </plugin>
-      </visual>
     </gazebo>
     <!-- LIGHT -->
