Commit message: road_description: updated circuit xacro files structure and launchs

File: road_description/urdf/trafficlight/trafficlight_macro.xacro (robot description, xacro)
@@ -3,13 +3,13 @@
   <xacro:include filename="$(find road_description)/urdf/materials.xacro" />
   <xacro:property name="PI" value="3.1415926535897931" />
-  <xacro:property name="panel_width"    value="0.08" />
+  <xacro:property name="panel_width"    value="0.06" />
   <xacro:property name="panel_depth"    value="0.03" />
   <xacro:property name="panel_height"   value="0.15" />
-  <xacro:property name="tag_size"       value="0.06" />
-  <xacro:property name="tag_z_offset"   value="0.03" />
+  <xacro:property name="tag_size"       value="0.05" />
+  <xacro:property name="tag_z_offset"   value="0.065" />
   <xacro:property name="delta"          value="0.001" />
-  <xacro:property name="light_width"    value="0.06" />
-  <xacro:property name="light_height"   value="0.03" />
-  <xacro:property name="light_z_offset" value="0.11" />
+  <xacro:property name="light_width"    value="0.05" />
+  <xacro:property name="light_height"   value="0.02" />
+  <xacro:property name="light_z_offset" value="0.13" />
   <xacro:macro name="trafficlight"
                params="name:=trafficlight

Commit message: Fixed color_plugin to work also with 16.04/kinetic (sdf issue)

File: road_description/urdf/trafficlight/trafficlight_macro.xacro (robot description, xacro)
@@ -1,4 +1,4 @@
 <?xml version="1.0"?>
-<root xmlns:xacro="http://ros.org/wiki/xacro">
+<root xmlns:xacro="http://www.ros.org/wiki/xacro">
   <xacro:include filename="$(find road_description)/urdf/materials.xacro" />
   <xacro:property name="PI" value="3.1415926535897931" />
@@ -118,7 +118,8 @@
       <visual>
         <plugin name="${name}_color_plugin" filename="libcolor_plugin.so" >
-          <element_name>${name}</element_name>
-          <material>${light_material}</material>
-          <material2>${light_material2}</material2>
+          <sdf>
+            <material>${light_material}</material>
+            <material2>${light_material2}</material2>
+          </sdf>
         </plugin>
       </visual>
